File: MatrixMixer.sch (KiCad schematic (older format))
At the start: 42 parts

Commit message: doc update
Parts:
- gave numbers to parts that had none: 39
Connections:
- net GND: now also U1.5 (+), U3.5 (+); no longer U1.3 (+), U3.3 (+)
- net at R11.2, RV4.1, RV4.3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: now also U1.6 (-); no longer U1.2 (-)
- net at R11.1, R14.2: now also U1.7; no longer U1.1
- net at J6.1 (TIP), R18.1: now also U3.7; no longer U3.1
- net at R15.1, R18.2, SW3.1 (A): now also U3.6 (-); no longer U3.2 (-)
